File: misc.sch (KiCad schematic (older format))
At the start: 13 parts, among them J3 USB_OTG, U4 RT9193-28, U5 AP7313-33SAG

Commit message: adding v2 2 filter front end filter
Parts:
- added JP2: 5V USB, Jumper:SolderJumper-2_P1.3mm_Open_RoundedPad1.0x1.5mm, symbol Jumper:SolderJumper_2_Open
- L2, L3, L4: value L -> 15uH; footprint Inductor_SMD:L_0805_2012Metric -> Inductor_SMD:L_1210_3225Metric
- renumbered U4 to U6, U5 to U7
Connections:
- net +5V: now also JP2.1 (A); no longer J3.1 (Pin_1)
- new net: J3.1 (Pin_1), JP2.2 (B)
Changed lines of the file:
@@
 encoding utf-8
 Sheet 5 5
-Title ""
+Title "AfriCUBE Satellite"
 Date ""
-Rev ""
-Comp ""
-Comment1 ""
+Rev "Version 1.0"
+Comp "GigaTechnology / AMSATSA"
+Comment1 "Anton Janovsky  Shahn Pretorius"
 Comment2 ""
 Comment3 ""
@@
 $EndDescr
 $Comp
-L power:GND #PWR057
+L power:GND #PWR061
 U 1 1 5C690F71
 P 4850 4050
-F 0 "#PWR057" H 4850 3800 50  0001 C CNN
+F 0 "#PWR061" H 4850 3800 50  0001 C CNN
 F 1 "GND" H 4850 3900 50  0000 C CNN
 F 2 "" H 4850 4050 50  0001 C CNN
@@
 $EndComp
 $Comp
-L power:GND #PWR056
+L power:GND #PWR060
 U 1 1 5C690F9B
 P 5200 4000
-F 0 "#PWR056" H 5200 3750 50  0001 C CNN
+F 0 "#PWR060" H 5200 3750 50  0001 C CNN
 F 1 "GND" H 5200 3850 50  0000 C CNN
 F 2 "" H 5200 4000 50  0001 C CNN
@@
 USB_DP
 $Comp
-L power:GND #PWR051
+L power:GND #PWR055
 U 1 1 5C6911FA
 P 4600 3200
-F 0 "#PWR051" H 4600 2950 50  0001 C CNN
+F 0 "#PWR055" H 4600 2950 50  0001 C CNN
 F 1 "GND" H 4600 3050 50  0000 C CNN
 F 2 "" H 4600 3200 50  0001 C CNN
@@
 $EndComp
 $Comp
-L power:GND #PWR053
+L power:GND #PWR057
 U 1 1 5C691B40
 P 6800 3250
-F 0 "#PWR053" H 6800 3000 50  0001 C CNN
+F 0 "#PWR057" H 6800 3000 50  0001 C CNN
 F 1 "GND" H 6800 3100 50  0000 C CNN
 F 2 "" H 6800 3250 50  0001 C CNN
@@
 $EndComp
 $Comp
-L power:GND #PWR052
+L power:GND #PWR056
 U 1 1 5C692086
 P 6450 3200
-F 0 "#PWR052" H 6450 2950 50  0001 C CNN
+F 0 "#PWR056" H 6450 2950 50  0001 C CNN
 F 1 "GND" H 6450 3050 50  0000 C CNN
 F 2 "" H 6450 3200 50  0001 C CNN
@@
 $EndComp
 $Comp
-L power:GND #PWR054
+L power:GND #PWR058
 U 1 1 5C6920B8
 P 7150 3250
-F 0 "#PWR054" H 7150 3000 50  0001 C CNN
+F 0 "#PWR058" H 7150 3000 50  0001 C CNN
 F 1 "GND" H 7150 3100 50  0000 C CNN
 F 2 "" H 7150 3250 50  0001 C CNN
@@
 $EndComp
 $Comp
-L power:GND #PWR048
+L power:GND #PWR052
 U 1 1 5C69221A
 P 6150 2200
-F 0 "#PWR048" H 6150 1950 50  0001 C CNN
+F 0 "#PWR052" H 6150 1950 50  0001 C CNN
 F 1 "GND" H 6150 2050 50  0000 C CNN
 F 2 "" H 6150 2200 50  0001 C CNN
@@
 V18-SYNTH
 $Comp
-L power:GND #PWR047
+L power:GND #PWR051
 U 1 1 5C692712
 P 5350 2200
-F 0 "#PWR047" H 5350 1950 50  0001 C CNN
+F 0 "#PWR051" H 5350 1950 50  0001 C CNN
 F 1 "GND" H 5350 2050 50  0000 C CNN
 F 2 "" H 5350 2200 50  0001 C CNN
@@
 $EndComp
 $Comp
-L power:GND #PWR050
+L power:GND #PWR054
 U 1 1 5C693D92
 P 7875 2725
-F 0 "#PWR050" H 7875 2475 50  0001 C CNN
+F 0 "#PWR054" H 7875 2475 50  0001 C CNN
 F 1 "GND" H 7875 2575 50  0000 C CNN
 F 2 "" H 7875 2725 50  0001 C CNN
@@
 P 6800 2550
 AR Path="/5CB1DEB2" Ref="U?"  Part="1"
-AR Path="/5C68CE79/5CB1DEB2" Ref="U5"  Part="1"
-F 0 "U5" H 6650 2675 50  0000 C CNN
+AR Path="/5C68CE79/5CB1DEB2" Ref="U7"  Part="1"
+F 0 "U7" H 6650 2675 50  0000 C CNN
 F 1 "AP7313-33SAG" H 6400 2750 50  0000 L CNN
 F 2 "Package_TO_SOT_SMD:SOT-23" H 6800 2775 50  0001 C CIN
@@
 $EndComp
 $Comp
-L msisdr-rescue:APE8865Y5-28-HF-3 U4
+L msisdr-rescue:APE8865Y5-28-HF-3 U6
 U 1 1 5CB1E3FD
 P 6150 1650
-F 0 "U4" H 5900 1875 50  0000 C CNN
+F 0 "U6" H 5900 1875 50  0000 C CNN
 F 1 "RT9193-28" H 6075 1875 50  0000 L CNN
 F 2 "Package_TO_SOT_SMD:SOT-23-5" H 6150 1975 50  0001 C CIN
@@
 $EndComp
 $Comp
-L power:GND #PWR049
+L power:GND #PWR053
 U 1 1 5CB1E8F3
 P 5700 2350
-F 0 "#PWR049" H 5700 2100 50  0001 C CNN
+F 0 "#PWR053" H 5700 2100 50  0001 C CNN
 F 1 "GND" H 5700 2200 50  0000 C CNN
 F 2 "" H 5700 2350 50  0001 C CNN
@@
 Connection ~ 7875 3200
 Wire Wire Line
-	7450 3500 7800 3500
+	7450 3500 7475 3500
 Wire Wire Line
 	5000 3800 7625 3800
@@
 $EndComp
 $Comp
-L power:+5V #PWR055
+L power:+5V #PWR059
 U 1 1 601FC1D1
 P 7450 3500
-F 0 "#PWR055" H 7450 3350 50  0001 C CNN
+F 0 "#PWR059" H 7450 3350 50  0001 C CNN
 F 1 "+5V" H 7465 3673 50  0000 C CNN
 F 2 "" H 7450 3500 50  0001 C CNN
 F 3 "" H 7450 3500 50  0001 C CNN
 	1    7450 3500
-	-1   0    0    1
-$EndComp
-Connection ~ 7450 3500
+	0    -1   -1   0
+$EndComp
 $Comp
 L Device:L L2
@@
 P 4975 1500
 F 0 "L2" V 5165 1500 50  0000 C CNN
-F 1 "L" V 5074 1500 50  0000 C CNN
-F 2 "Inductor_SMD:L_0805_2012Metric" H 4975 1500 50  0001 C CNN
+F 1 "15uH" V 5074 1500 50  0000 C CNN
+F 2 "Inductor_SMD:L_1210_3225Metric" H 4975 1500 50  0001 C CNN
 F 3 "~" H 4975 1500 50  0001 C CNN
 	1    4975 1500
@@
 P 5725 2650
 F 0 "L3" V 5600 2650 50  0000 C CNN
-F 1 "L" V 5675 2650 50  0000 C CNN
-F 2 "Inductor_SMD:L_0805_2012Metric" H 5725 2650 50  0001 C CNN
+F 1 "15uH" V 5675 2650 50  0000 C CNN
+F 2 "Inductor_SMD:L_1210_3225Metric" H 5725 2650 50  0001 C CNN
 F 3 "~" H 5725 2650 50  0001 C CNN
 	1    5725 2650
@@
 P 7450 2900
 F 0 "L4" H 7502 2946 50  0000 L CNN
-F 1 "L" H 7502 2855 50  0000 L CNN
-F 2 "Inductor_SMD:L_0805_2012Metric" H 7450 2900 50  0001 C CNN
+F 1 "15uH" H 7502 2855 50  0000 L CNN
+F 2 "Inductor_SMD:L_1210_3225Metric" H 7450 2900 50  0001 C CNN
 F 3 "~" H 7450 2900 50  0001 C CNN
 	1    7450 2900
 	1    0    0    -1
 $EndComp
+$Comp
+L Jumper:SolderJumper_2_Open JP2
+U 1 1 6023965F
+P 7625 3500
+F 0 "JP2" H 7625 3400 50  0000 C CNN
+F 1 "5V USB" H 7300 3425 50  0000 C CNN
+F 2 "Jumper:SolderJumper-2_P1.3mm_Open_RoundedPad1.0x1.5mm" H 7625 3500 50  0001 C CNN
+F 3 "~" H 7625 3500 50  0001 C CNN
+	1    7625 3500
+	1    0    0    -1
+$EndComp
+Wire Wire Line
+	7775 3500 7800 3500
 Wire Wire Line
 	7450 3050 7450 3500
+Connection ~ 7450 3500
 $EndSCHEMATC
